Commit message: 10.09 MTC Test_Obstacle_Planner anepasst

File: install/estun_description/share/estun_description/urdf/estun.xacro (robot description, xacro)
@@ -142,4 +142,11 @@
     </geometry>
   </collision>
+</link>
+<link name= "estun_hand">
+  <inertial>
+    <origin xyz="0 0 0" rpy="0 0 0"/>
+    <mass value="0.1"/>
+    <inertia ixx="0.001" iyy="0.001" izz="0.001" ixy="0.0" iyz="0.0" ixz="0.0001"/>
+  </inertial>
 </link>
 <joint name="Umdrehung 1" type="continuous">
@@ -186,8 +193,15 @@
 </joint>
 <joint name="world_base_link" type="fixed">
-  <origin xyz="0 0 0" rpy="0 0 0"/>
+  <origin xyz="-0.2 0 0" rpy="0 0 0"/>
   <parent link="world"/>
   <child link="base_link"/>
   <axis xyz="0 0 0"/>
 </joint>
+<joint name="hand_endeffector_1" type="continuous">
+  <origin xyz="0 0 0" rpy="0 0 0"/>
+  <parent link="endeffector_1"/>
+  <child link="estun_hand"/>
+  <axis xyz="0 0 1"/>
+  <limit effort="1000.0" lower="-3.14" upper="3.14" velocity="10.0"/>
+</joint>
 </robot>

File: install/estun_moveit/share/estun_moveit/urdf/estun.ros2_control.xacro (robot description, xacro)
@@ -51,4 +51,10 @@
                 <state_interface name="velocity"/>
             </joint>
+            <joint name="hand_endeffector_1">
+                <command_interface name="position"/>
+                <state_interface name="position">
+                </state_interface>
+                <state_interface name="velocity"/>
+            </joint>
         </ros2_control>
         <gazebo>

Commit message: Pick and Place funktional für Dummy 11.11

File: install/estun_description/share/estun_description/urdf/estun.xacro (robot description, xacro)
@@ -198,10 +198,10 @@
   <axis xyz="0 0 0"/>
 </joint>
-<joint name="hand_endeffector_1" type="continuous">
-  <origin xyz="0 0 0" rpy="0 0 0"/>
+<joint name="hand_endeffector_1" type="prismatic">
+  <origin xyz="-0.1 0 0" rpy="0 0 0"/>
   <parent link="endeffector_1"/>
   <child link="estun_hand"/>
-  <axis xyz="0 0 1"/>
-  <limit effort="1000.0" lower="-3.14" upper="3.14" velocity="10.0"/>
+  <axis xyz="1 0 0"/>
+  <limit effort="1000.0" lower="0.0" upper="0.2" velocity="10.0"/>
 </joint>
 </robot>

File: install/estun_moveit/share/estun_moveit/urdf/estun.ros2_control.xacro (robot description, xacro)
@@ -52,5 +52,5 @@
             </joint>
             <joint name="hand_endeffector_1">
-                <command_interface name="position"/>
+                <!-- <command_interface name="position"/> -->
                 <state_interface name="position">
                 </state_interface>
