Commit message: MTC funktioniert 26.10

File: src/estun_description/urdf/estun.xacro (robot description, xacro)
@@ -143,5 +143,12 @@
   </collision>
 </link>
-<link name= "estun_hand">
+<link name= "estun_hand_0">
+  <inertial>
+    <origin xyz="0 0 0" rpy="0 0 0"/>
+    <mass value="0.1"/>
+    <inertia ixx="0.001" iyy="0.001" izz="0.001" ixy="0.0" iyz="0.0" ixz="0.0001"/>
+  </inertial>
+</link>
+<link name= "estun_hand_1">
   <inertial>
     <origin xyz="0 0 0" rpy="0 0 0"/>
@@ -198,8 +205,14 @@
   <axis xyz="0 0 0"/>
 </joint>
-<joint name="hand_endeffector_1" type="prismatic">
+<joint name="hand_endeffector_0" type="fixed">
   <origin xyz="-0.1 0 0" rpy="0 0 0"/>
   <parent link="endeffector_1"/>
-  <child link="estun_hand"/>
+  <child link="estun_hand_0"/>
+  <axis xyz="1 0 0"/>
+</joint>
+<joint name="hand_endeffector_1" type="continuous">
+  <origin xyz="-0.1 0 0" rpy="0 0 0"/>
+  <parent link="estun_hand_0"/>
+  <child link="estun_hand_1"/>
   <axis xyz="1 0 0"/>
   <limit effort="1000.0" lower="0.0" upper="0.2" velocity="10.0"/>

File: src/estun_moveit/urdf/estun.ros2_control.xacro (robot description, xacro)
@@ -52,5 +52,5 @@
             </joint>
             <joint name="hand_endeffector_1">
-                <!-- <command_interface name="position"/> -->
+                <command_interface name="position"/>
                 <state_interface name="position">
                 </state_interface>
